Commit message: Conversion of robot meshes to obj files to be better compatible with unity

File: data/franka_panda/robot.urdf (robot description, URDF)
Before this commit: robot panda, 17 links, 16 joints
Links:
- link panda_link0: geometry collision mesh filename=package://franka_description/meshes/collision/link0.stl; visual mesh filename=/meshes/link0.obj
- link panda_link1: geometry collision mesh filename=package://franka_description/meshes/collision/link1.stl; visual mesh filename=/meshes/link1.obj
- link panda_link2: geometry collision mesh filename=package://franka_description/meshes/collision/link2.stl; visual mesh filename=/meshes/link2.obj
- link panda_link3: geometry collision mesh filename=package://franka_description/meshes/collision/link3.stl; visual mesh filename=/meshes/link3.obj
- link panda_link4: geometry collision mesh filename=package://franka_description/meshes/collision/link4.stl; visual mesh filename=/meshes/link4.obj
- link panda_link5: geometry collision mesh filename=package://franka_description/meshes/collision/link5.stl; visual mesh filename=/meshes/link5.obj
- link panda_link6: geometry collision mesh filename=package://franka_description/meshes/collision/link6.stl; visual mesh filename=/meshes/link6.obj
- link panda_link7: geometry collision mesh filename=package://franka_description/meshes/collision/link7.stl; visual mesh filename=/meshes/link7.obj

File: data/kinova_gen3/robot.urdf (robot description, URDF)
Before this commit: robot kinovagen3, 13 links, 12 joints
Links:
- link base_link: geometry collision mesh filename=/meshes/base_link.obj; visual mesh filename=/meshes/base_link.obj
- link bracelet_link: geometry collision mesh filename=/meshes/bracelet_with_vision_link.obj; visual mesh filename=/meshes/bracelet_with_vision_link.obj
- link forearm_link: geometry collision mesh filename=/meshes/forearm_link.obj; visual mesh filename=/meshes/forearm_link.obj
- link half_arm_1_link: geometry collision mesh filename=/meshes/half_arm_1_link.obj; visual mesh filename=/meshes/half_arm_1_link.obj
- link half_arm_2_link: geometry collision mesh filename=/meshes/half_arm_2_link.obj; visual mesh filename=/meshes/half_arm_2_link.obj
- link shoulder_link: geometry collision mesh filename=/meshes/shoulder_link.obj; visual mesh filename=/meshes/shoulder_link.obj
- link spherical_wrist_1_link: geometry collision mesh filename=/meshes/spherical_wrist_1_link.obj; visual mesh filename=/meshes/spherical_wrist_1_link.obj
- link spherical_wrist_2_link: geometry collision mesh filename=/meshes/spherical_wrist_2_link.obj; visual mesh filename=/meshes/spherical_wrist_2_link.obj

File: data/robotiq_2f85gripper/robot.urdf (robot description, URDF)
Before this commit: robot robotiq_arg85, 9 links, 8 joints
Links:
- link left_inner_finger: geometry collision mesh filename=/meshes/inner_finger_coarse.obj; visual mesh filename=/meshes/inner_finger_fine.obj
- link left_inner_knuckle: geometry collision mesh filename=/meshes/inner_knuckle_coarse.obj; visual mesh filename=/meshes/inner_knuckle_fine.obj
- link left_outer_finger: geometry collision mesh filename=/meshes/outer_finger_coarse.obj
- link left_outer_knuckle: geometry collision mesh filename=/meshes/outer_knuckle_coarse.obj; visual mesh filename=/meshes/outer_finger_fine.obj
- link right_inner_finger: geometry collision mesh filename=/meshes/inner_finger_coarse.obj; visual mesh filename=/meshes/inner_finger_fine.obj
- link right_inner_knuckle: geometry collision mesh filename=/meshes/inner_knuckle_coarse.obj; visual mesh filename=/meshes/inner_knuckle_fine.obj
- link right_outer_finger: geometry collision mesh filename=/meshes/outer_finger_coarse.obj
- link right_outer_knuckle: geometry collision mesh filename=/meshes/outer_knuckle_coarse.obj; visual mesh filename=/meshes/outer_finger_fine.obj
- link robotiq_85_base_link: geometry collision mesh filename=/meshes/robotiq_85_base_link_coarse.obj; visual mesh filename=/meshes/robotiq_85_base_link_fine.obj
