Commit message: Replaced yumi meshes with simplified versions

File: data/bd_spot_base/floating_base.urdf (robot description, URDF)
Before this commit: robot spot_floating_base, 1 links, 0 joints
Links:
- link body: geometry 

Commit message: Added cube mesh for spot base agent robot

File: data/bd_spot_base/floating_base.urdf (robot description, URDF)
Before this commit: robot spot_floating_base, 1 links, 0 joints
Links:
- link body: geometry visual mesh filename=/meshes/cube.obj scale=0.4 0.2 0.1
