Commit message: Converted robot tests into unit tests

File: source/apps/config/test_robots/testRobot2.urdf (robot description, URDF)
Before this commit: robot dummy, 11 links, 10 joints
Links:
- removed link base
- added link link0
Joints:
- joint joint1: parent base -> link0
- joint joint2: parent base -> link0
